Commit message: transition from 4-wheeled robot to 2-wheeled robot+ a support caster wheel

File: src/wayfinder_description/urdf/ros2_control.xacro (robot description, xacro)
@@ -10,9 +10,9 @@
             <command_interface name="velocity"/>
         </joint>
-        <joint name="rear_left_wheel_joint">
+        <!-- <joint name="rear_left_wheel_joint">
             <state_interface name="position"/>
             <state_interface name="velocity"/>
             <command_interface name="velocity"/>
-        </joint>
+        </joint> -->
         <joint name="front_right_wheel_joint">
             <state_interface name="position"/>
@@ -20,9 +20,9 @@
             <command_interface name="velocity"/>
         </joint>
-        <joint name="rear_right_wheel_joint">
+        <!-- <joint name="rear_right_wheel_joint">
             <state_interface name="position"/>
             <state_interface name="velocity"/>
             <command_interface name="velocity"/>
-        </joint>
+        </joint> -->
     </ros2_control>
     <gazebo>

File: src/wayfinder_description/urdf/wayfinder.urdf.xacro (robot description, xacro)
@@ -27,6 +27,35 @@
     <xacro:wheel prefix="front_left"  x_offset="0.18"  y_offset="0.21"/>
     <xacro:wheel prefix="front_right" x_offset="0.18"  y_offset="-0.21"/>
-    <xacro:wheel prefix="rear_left"   x_offset="-0.18" y_offset="0.21"/>
-    <xacro:wheel prefix="rear_right"  x_offset="-0.18" y_offset="-0.21"/>
+    <!--
+        <xacro:wheel prefix="rear_left"   x_offset="-0.18" y_offset="0.21"/>
+        <xacro:wheel prefix="rear_right"  x_offset="-0.18" y_offset="-0.21"/>
+    -->
+    <link name="caster_wheel_link">
+        <visual>
+            <geometry>
+                <sphere radius="0.04"/>
+            </geometry>
+            <material name="black"/>
+        </visual>
+        <collision>
+            <geometry>
+                <sphere radius="0.04"/>
+            </geometry>
+        </collision>
+        <inertial>
+            <origin xyz="0 0 0" rpy="0 0 0"/>
+            <mass value="0.1"/>
+            <inertia ixx="0.000064" iyy="0.000064" izz="0.000064" ixy="0" ixz="0" iyz="0"/>
+        </inertial>
+    </link>
+    <joint name="caster_wheel_joint" type="fixed">
+        <parent link="base_link"/>
+        <child link="caster_wheel_link"/>
+        <origin xyz="-0.18 0 -0.09" rpy="0 0 0"/>
+    </joint>
+    <gazebo reference="caster_wheel_link">
+        <mu1>0.0</mu1>
+        <mu2>0.0</mu2>
+    </gazebo>
     <xacro:include filename="$(find wayfinder_description)/urdf/sensors.xacro"/>
     <xacro:include filename="$(find wayfinder_description)/urdf/ros2_control.xacro"/>
