Commit message: add camera to the robot

File: src/wayfinder_description/urdf/sensors.xacro (robot description, xacro)
@@ -44,4 +44,42 @@
         </sensor>
     </gazebo>
-    <!-- TODO camera link, joint -->
+    <link name="camera_link">
+        <visual>
+            <geometry><box size="0.03 0.06 0.03"/></geometry>
+            <material name="black"/>
+        </visual>
+        <collision>
+            <geometry><box size="0.03 0.06 0.03"/></geometry>
+        </collision>
+        <inertial>
+            <origin xyz="0 0 0" rpy="0 0 0"/>
+            <mass value="0.05"/>
+            <inertia ixx="0.00002" iyy="0.00001" izz="0.00002" ixy="0" ixz="0" iyz="0"/>
+        </inertial>
+    </link>
+    <joint name="camera_joint" type="fixed">
+        <parent link="base_link"/>
+        <child link="camera_link"/>
+        <origin xyz="0.22 0 0.08" rpy="0 0 0"/>
+    </joint>
+    <gazebo reference="camera_link">
+        <sensor name="camera_sensor" type="camera">
+            <update_rate>15</update_rate>
+            <topic>camera/image_raw</topic>
+            <gz_frame_id>camera_link</gz_frame_id>
+            <visualize>true</visualize>
+            <camera>
+                <horizontal_fov>1.3</horizontal_fov>
+                <image>
+                    <width>640</width>
+                    <height>480</height>
+                    <format>R8G8B8</format>
+                </image>
+                <clip>
+                    <near>0.05</near>
+                    <far>20.0</far>
+                </clip>
+            </camera>
+        </sensor>
+    </gazebo>
  </robot>
